File: eagle/pulseGeneratorArduinoV1.1.brd (EAGLE design)
At the start: 100 x 80 mm, 6 parts, among them U1 ARDUINOR3-DIMENSION, U2 AD9954YSVZ, U3 TXB0104PWR, U4 LT1962EMS8-1.8PBF, U5 LT1962EMS8-1.8PBF

Commit message: made progress
Parts:
- added C1, C10, C11, C12, C14, C2, C3, C4, C5, C6, C7, C8, C9: 0.1uF, resistor:C0402
- added C13: 1uF, resistor:C0402
- added C15, C16: 1nF, resistor:C0402
- added C17, C20, C21: 10nF, resistor:C0402
- added C18, C19: 4.7uF, resistor:C0402
- added C22, C23: 10uF, resistor:C0402
- added L1, L2: (no value), SparkFun-Passives:0603
- added R1, R3: 0, resistor:R0402
- added R2: 3.92K, resistor:R0402
- added R4: 100, resistor:R0402
Connections:
- removed net 3V: U1.3V
- removed net AVDD: U2.16
- removed net AVDD_2: U2.6
- removed net AVDD_3: U2.13
- removed net AVDD_4: U2.18
- removed net AVDD_5: U2.4
- removed net AVDD_6: U2.29
- removed net AVDD_7: U2.19
- removed net AVDD_8: U2.27
- removed net AVDD_9: U2.25
- removed net DVDD: U2.34
- removed net DVDD_2: U2.2
- removed net DVDD_I/O: U2.43
- removed net IN: U4.8, U5.8
- new net *COMPIN: U2.31
- new net *IOUT: U2.20
- new net *OSC: C15.2, U2.8
- new net COMPIN: U2.30
- new net CRYSTALOUT: U2.10
- new net GNDA: C10.2, C11.2, C12.2, C13.2, C18.2, C19.2, C20.2, C21.2, C22.2, C23.2, C4.2, C5.2, C6.2, C7.2, C8.2, C9.2, R2.1, U2.14, U2.15, U2.17, U2.22, U2.26, U2.32, U2.49, U2.5, U2.7, U4.4, U5.4
- new net MISO: U2.38
- new net MOSI: U2.41
- new net N$1: C14.1, R1.1
- new net N$11: C17.1, U$1.6
- new net N$12: C22.1, L2.1, U5.5, U5.8
- new net N$13: C23.1, L1.1, U4.5, U4.8
- new net N$14: C20.1, U5.3
- new net N$15: C21.1, U4.3
- new net N$18: L1.2, L2.2, U1.3V
- new net N$2: C16.1, R4.1, U$1.4
- new net N$3: R3.2, U2.44
- new net N$5: C15.1, R4.2, U$1.5
- new net N$6: R1.2, U2.12
- new net N$7: C13.1, U2.23
- new net N$8: R2.2, U2.24
- new net N$9: U2.28
- new net OSC: C16.2, U2.9
- new net OSK: U2.46
- new net OUT: U2.21
- new net PS0: U2.47
- new net PS1: U2.48
- new net RESET: U2.36
- new net SCLK: U2.40
- new net SS: U2.37, U2.39
- new net SYNCCLK: U2.45
- new net UPDATE: U2.1
- new net VSS: C10.1, C11.1, C12.1, C18.1, C4.1, C5.1, C6.1, C7.1, C8.1, C9.1, U2.13, U2.16, U2.18, U2.19, U2.25, U2.27, U2.29, U2.4, U2.6, U4.1, U4.2
- net GND: now also C1.2, C17.2, C2.2, C3.2, R3.1, U$1.3, U2.11, U2.3, U2.33, U2.35, U2.42
- net VDD: now also C1.1, C14.2, C19.1, C2.1, C3.1, U2.2, U2.34, U2.43, U5.1, U5.2; no longer U$1.6
