File: eagle/pulseGeneratorArduinoV1.1.sch (EAGLE design)
At the start: 6 parts, among them U1 ARDUINOR3-DIMENSION, U2 AD9954YSVZ, U3 TXB0104PWR, U4 LT1962EMS8-1.8PBF, U5 LT1962EMS8-1.8PBF

Commit message: made progress
Parts:
- added C1, C10, C11, C12, C14, C2, C3, C4, C5, C6, C7, C8, C9: 0.1uF, resistor:C-USC0402
- added C13: 1uF, resistor:C-USC0402
- added C15, C16: 1nF, resistor:C-USC0402
- added C17, C20, C21: 10nF, resistor:C-USC0402
- added C18, C19: 4.7uF, resistor:C-USC0402
- added C22, C23: 10uF, resistor:C-USC0402
- added L1, L2: (no value), SparkFun-Passives:INDUCTOR0603
- added R1, R3: 0, resistor:R-US_R0402
- added R2: 3.92K, resistor:R-US_R0402
- added R4: 100, resistor:R-US_R0402
Connections:
- new net *COMPIN: U2.~COMP_IN
- new net *IOUT: U2.~IOUT
- new net *OSC: C15.2, U2.~OSC/~REFCLK
- new net COMPIN: U2.COMP_IN
- new net CRYSTALOUT: U2.CRYSTAL_OUT
- new net GND: C1.2, C17.2, C2.2, C3.2, R3.1, U$1.GND, U2.CLKMODESELECT, U2.DGND, U2.DGND_2, U2.DGND_3, U2.PWRDWNCTL
- new net GNDA: C10.2, C11.2, C12.2, C13.2, C18.2, C19.2, C20.2, C21.2, C22.2, C23.2, C4.2, C5.2, C6.2, C7.2, C8.2, C9.2, R2.1, U2.AGND, U2.AGND_2, U2.AGND_3, U2.AGND_4, U2.AGND_5, U2.AGND_6, U2.AGND_7, U2.AGND_8, U2.EPAD, U4.GND, U5.GND
- new net MISO: U2.SDO
- new net MOSI: U2.SDIO
- new net N$1: C14.1, R1.1
- new net N$11: C17.1, U$1.VDD
- new net N$12: C22.1, L2.1, U5.IN, U5.~SHDN
- new net N$13: C23.1, L1.1, U4.IN, U4.~SHDN
- new net N$14: C20.1, U5.BYP
- new net N$15: C21.1, U4.BYP
- new net N$18: L1.2, L2.2, U1.3V
- new net N$2: C16.1, R4.1, U$1.CLK
- new net N$3: R3.2, U2.SYNC_IN
- new net N$5: C15.1, R4.2, U$1.*CLK
- new net N$6: R1.2, U2.LOOP_FILTER
- new net N$7: C13.1, U2.DACBP
- new net N$8: R2.2, U2.DAC_RSET
- new net N$9: U2.COMP_OUT
- new net OSC: C16.2, U2.OSC/REFCLK
- new net OSK: U2.OSK
- new net OUT: U2.IOUT
- new net PS0: U2.PS0
- new net PS1: U2.PS1
- new net RESET: U2.RESET
- new net SCLK: U2.SCLK
- new net SS: U2.IOSYNC, U2.~CS
- new net SYNCCLK: U2.SYNC_CLK
- new net UPDATE: U2.I/O_UPDATE
- new net VDD: C1.1, C14.2, C19.1, C2.1, C3.1, U2.DVDD, U2.DVDD_2, U2.DVDD_I/O, U5.OUT, U5.SENSE
- new net VSS: C10.1, C11.1, C12.1, C18.1, C4.1, C5.1, C6.1, C7.1, C8.1, C9.1, U2.AVDD, U2.AVDD_2, U2.AVDD_3, U2.AVDD_4, U2.AVDD_5, U2.AVDD_6, U2.AVDD_7, U2.AVDD_8, U2.AVDD_9, U4.OUT, U4.SENSE
Other:
- moved on the sheet: U3, U4, U5
